Commit message: fix collision parameter and remove unused file

File: su065d4380_description/urdf/common/constants.xacro (robot description, xacro)
@@ -1,7 +1,4 @@
 <?xml version="1.0" encoding="UTF-8"?>
 <robot xmlns:xacro="http://ros.org/wiki/xacro">
-  <xacro:property
-      name="SCALE_MM"
-      value="0.001" />
   <xacro:property
       name="PI"

File: su065d4380_description/urdf/su065d4380.xacro (robot description, xacro)
@@ -7,10 +7,4 @@
       filename="$(find su065d4380_description)/urdf/common/constants.xacro"
       ns="const" />
-  <xacro:property
-      name="wheel_col_len"
-      value="0.055" />
-  <xacro:property
-      name="wheel_col_radius"
-      value="0.075" /> <!-- = 0.0785/2 -->
   <xacro:macro
       name="su065d4380"
@@ -42,13 +36,12 @@
         <origin
             xyz="0 0 0"
-            rpy="0 0 0" />
+            rpy="${90.0 * const.TO_RADIAN} 0 0" />
         <geometry>
           <cylinder
-              length="${wheel_col_len}"
-              radius="${wheel_col_radius}" />
+              length="45.0e-3"
+              radius="75.0e-3" />
         </geometry>
       </collision>
     </link>
-    <!-- wheel offset is 18iuse_nominal_extrinsics} -->
     <link name="${prefix}su065d4380_wheel_motor_link">
       <inertial>
@@ -75,12 +68,21 @@
       <collision>
         <origin
-            xyz="0 0 0"
-            rpy="0 0 0" />
+            xyz="0 -89.75e-3 0"
+            rpy="${-90.0 * const.TO_RADIAN} 0 0" />
         <geometry>
-          <box size="0 0 0" />
+          <cylinder
+              length="205.50e-3"
+              radius="30.08e-3" />
         </geometry>
       </collision>
     </link>
     <!-- Joints -->
+    <joint
+        name="${prefix}su065d4380_joint"
+        type="fixed">
+      <parent link="${parent}" />
+      <child link="${prefix}su065d4380_wheel_motor_link" />
+      <xacro:insert_block name="origin" />
+    </joint>
     <joint
         name="${prefix}su065d4380_wheel_joint"
@@ -91,18 +93,6 @@
       <axis xyz="0 1 0" />
       <origin
-          xyz="0 0.018 0"
+          xyz="0 40.5e-3 0"
           rpy="0 0 0" />
-      <limit
-          effort="30"
-          velocity="1.0"
-          lower="-2.2"
-          upper="0.7" />
-    </joint>
-    <joint
-        name="${prefix}su065d4380_joint"
-        type="fixed">
-      <parent link="${parent}" />
-      <child link="${prefix}su065d4380_wheel_motor_link" />
-      <xacro:insert_block name="origin" />
     </joint>
   </xacro:macro>
