Commit message: fix component order to make it consistent with the tree structure

File: su065d4380_description/urdf/su065d4380.xacro (robot description, xacro)
@@ -11,4 +11,37 @@
       params="parent prefix *origin">
     <!-- Link -->
+    <link name="${prefix}su065d4380_wheel_motor_link">
+      <inertial>
+        <origin
+            xyz="0 0 0"
+            rpy="0 0 0" />
+        <mass value="1.105" />
+        <inertia
+            ixx=".000285"
+            ixy="0.0"
+            ixz="0.0"
+            iyy="0.00286"
+            iyz="0.0"
+            izz="0.00285" />
+      </inertial>
+      <visual>
+        <origin
+            xyz="0 0 0"
+            rpy="0 0 0" />
+        <geometry>
+          <mesh filename="package://su065d4380_description/meshes/wheel_motor.dae" />
+        </geometry>
+      </visual>
+      <collision>
+        <origin
+            xyz="0 -89.75e-3 0"
+            rpy="${-90.0 * const.TO_RADIAN} 0 0" />
+        <geometry>
+          <cylinder
+              length="205.50e-3"
+              radius="30.08e-3" />
+        </geometry>
+      </collision>
+    </link>
     <link name="${prefix}su065d4380_wheel_link">
       <inertial>
@@ -44,37 +77,4 @@
       </collision>
     </link>
-    <link name="${prefix}su065d4380_wheel_motor_link">
-      <inertial>
-        <origin
-            xyz="0 0 0"
-            rpy="0 0 0" />
-        <mass value="1.105" />
-        <inertia
-            ixx=".000285"
-            ixy="0.0"
-            ixz="0.0"
-            iyy="0.00286"
-            iyz="0.0"
-            izz="0.00285" />
-      </inertial>
-      <visual>
-        <origin
-            xyz="0 0 0"
-            rpy="0 0 0" />
-        <geometry>
-          <mesh filename="package://su065d4380_description/meshes/wheel_motor.dae" />
-        </geometry>
-      </visual>
-      <collision>
-        <origin
-            xyz="0 -89.75e-3 0"
-            rpy="${-90.0 * const.TO_RADIAN} 0 0" />
-        <geometry>
-          <cylinder
-              length="205.50e-3"
-              radius="30.08e-3" />
-        </geometry>
-      </collision>
-    </link>
     <!-- Joints -->
     <joint

Commit message: Fix inertial and mass

File: su065d4380_description/urdf/su065d4380.xacro (robot description, xacro)
@@ -14,14 +14,14 @@
       <inertial>
         <origin
-            xyz="0 0 0"
+            xyz="0 -68.0e-3 0"
             rpy="0 0 0" />
-        <mass value="1.105" />
+        <mass value="3.27" />
         <inertia
-            ixx=".000285"
+            ixx="0.03"
             ixy="0.0"
             ixz="0.0"
-            iyy="0.00286"
+            iyy="0.003"
             iyz="0.0"
-            izz="0.00285" />
+            izz="0.03" />
       </inertial>
       <visual>
@@ -49,12 +49,12 @@
             xyz="0 0 0"
             rpy="0 0 0" />
-        <mass value="6.141" />
+        <mass value="3.63" />
         <inertia
-            ixx="0.00349"
+            ixx="0.006"
             ixy="0.0"
             ixz="0.0"
-            iyy="0.00630"
+            iyy="0.011"
             iyz="0.0"
-            izz="0.00349" />
+            izz="0.006" />
       </inertial>
       <visual>
